File: litl.kicad_pcb (KiCad board)
At the start: 2 copper layers, 100 parts, among them J1 Conn_01x04, SW1 KEYSW, SW10 KEYSW, SW11 KEYSW, SW12 KEYSW, SW13 KEYSW, SW14 KEYSW, SW15 KEYSW, SW16 KEYSW, SW17 KEYSW, SW18 KEYSW, SW19 KEYSW, SW2 KEYSW, SW20 KEYSW, SW21 KEYSW, SW22 KEYSW, SW23 KEYSW, SW24 KEYSW, SW25 KEYSW, SW26 KEYSW, SW27 KEYSW, SW28 KEYSW, SW29 KEYSW, SW3 KEYSW, SW30 KEYSW, SW31 KEYSW, SW32 KEYSW, SW33 KEYSW, SW34 KEYSW, SW35 KEYSW, SW36 KEYSW, SW37 KEYSW, SW38 KEYSW, SW39 KEYSW, SW4 KEYSW, SW40 KEYSW, SW41 KEYSW, SW42 KEYSW, SW43 KEYSW, SW44 KEYSW, SW45 KEYSW, SW46 KEYSW, SW47 KEYSW, SW48 KEYSW, SW49 KEYSW, SW5 KEYSW, SW50 KEYSW, SW51 RotaryEncoder_Switch, SW52 SW_PUSH, SW6 KEYSW, SW7 KEYSW, SW8 KEYSW, SW9 KEYSW, U1 ProMicro

Commit message: Footprints placed
Parts:
- SW15: footprint Button_Switch_Keyboard:SW_Cherry_MX_1.75u_PCB -> Button_Switch_Keyboard:SW_Cherry_MX_1.00u_PCB
- moved SW52 330.3 mm to (181.4, 21.5)
- moved D42 320.9 mm to (198.2, 38.2), turned to 90 degrees
- moved D46 306.1 mm to (202.9, 38.2), turned to 90 degrees
- moved D45 300.6 mm to (181.4, 38.2), turned to 90 degrees
- moved D36 299.7 mm to (164.7, 38.2), turned to 90 degrees
- moved D43 292.8 mm to (179.1, 38.2), turned to 90 degrees
- moved D28 291.7 mm to (155.2, 38.2), turned to 90 degrees
- moved D19 289.8 mm to (100.3, 35.8)
- moved D40 288.2 mm to (195.8, 38.2), turned to 90 degrees
- moved D16 286.5 mm to (88.3, 33.4)
- moved D15 285.6 mm to (100.3, 31.0)
- moved D32 285.3 mm to (160.0, 38.2), turned to 90 degrees
- moved D39 284.7 mm to (174.3, 38.2), turned to 90 degrees
- moved D27 284.6 mm to (136.1, 38.2), turned to 90 degrees
- moved SW13 283.8 mm to (262.8, 71.3)
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
Commit message: Diode layout complete
Parts:
- added D47: D_Small, Keebio-Parts:Diode, F.Cu at (193.4, 43.0)
- added SW53: RotaryEncoder_Switch, Keebio-Parts:RotaryEncoder_EC11, F.Cu at (234.2, 35.8)
- SW52: footprint Keebio-Parts:SW_Tactile_SPST_Angled_MJTP1117-no-mount -> Button_Switch_THT:SW_PUSH_6mm
- moved D11 122.6 mm to (186.2, 28.6)
- moved D12 122.6 mm to (198.2, 28.6)
- moved D38 119.5 mm to (74.0, 43.0), turned to 0 degrees
- moved D13 100.7 mm to (188.6, 33.4)
- moved D24 100.7 mm to (200.6, 33.4)
- moved D10 98.6 mm to (174.3, 28.6)
- moved D9 98.6 mm to (162.3, 28.6)
- moved D40 98.0 mm to (97.9, 43.0), turned to 0 degrees
- moved D39 88.5 mm to (86.0, 43.0), turned to 0 degrees
- moved D22 76.7 mm to (164.7, 33.4)
- moved D23 76.7 mm to (176.7, 33.4)
- moved D7 74.6 mm to (138.5, 28.6)
- moved D8 74.6 mm to (150.4, 28.6)
- moved SW52 73.2 mm to (112.2, 45.4), turned to 180 degrees
- moved D26 69.2 mm to (83.6, 38.2), turned to 0 degrees
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Connections:
- net +5V renamed GND
- D37 pad 1: rowG -> rowH
- D42 pad 1: rowG -> rowH
- D43 pad 1: rowH -> rowG
- D44 pad 1: rowH -> rowG
- D45 pad 1: rowG -> rowH
- SW41 pad 1: col3 -> col2
- SW42 pad 1: col4 -> col3
- SW47 pad 1: col3 -> col2
- SW50 pad 1: RotB -> col4
Other:
- board outline added: 253.1 x 102.7 mm

Commit message: Vias added
Parts:
- removed SW52: SW_PUSH, Button_Switch_THT:SW_PUSH_6mm
- moved D44 23.9 mm to (193.4, 43.0)
- moved D45 23.9 mm to (205.3, 43.0)
- moved D46 23.9 mm to (181.4, 43.0)
- moved D47 23.9 mm to (169.5, 43.0)
- moved SW41 0.05 mm to (145.8, 109.6)
- turned SW51 to -90 degrees
- turned SW53 to -90 degrees
Connections:
- U1 pad 22: RST -> unconnected-(U1-Pad22)
Routing:
- net col3: track 0.00 -> 167.7 mm
- net col4: track 0.00 -> 165.4 mm
- net col2: track 0.00 -> 153.1 mm
- net col0: track 0.00 -> 146.9 mm
- net RotB: track 0.00 -> 128.9 mm
- net col1: track 0.00 -> 128.9 mm
- net Net-(D45-Pad2): track 0.00 -> 124.8 mm
- net rowA: track 0.00 -> 124.1 mm
- net rowC: track 0.00 -> 124.1 mm
- net rowG: track 0.00 -> 124.1 mm
- net rowF: track 0.00 -> 124.1 mm
- net rowE: track 0.00 -> 124.1 mm
- net rowD: track 0.00 -> 124.1 mm
- net rowB: track 0.00 -> 124.1 mm
- net rowH: track 0.00 -> 123.2 mm
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Other:
- board size 253.1 x 102.7 mm -> 248.3 x 100.3 mm
- board text added: "litl v1"

Commit message: Tracks done
Parts:
- U1: moved to B.Cu
Connections:
- U1 pad 10: col3 -> rowF
- U1 pad 11: col4 -> rowA
- U1 pad 12: RotB -> rowB
- U1 pad 13: rowH -> RotB
- U1 pad 14: rowG -> col4
- U1 pad 15: rowF -> col3
- U1 pad 16: rowE -> col2
- U1 pad 17: rowD -> col1
- U1 pad 18: rowC -> col0
- U1 pad 19: rowB -> rowG
- U1 pad 20: rowA -> rowH
- U1 pad 7: col0 -> rowC
- U1 pad 8: col1 -> rowD
- U1 pad 9: col2 -> rowE
Routing:
- net GND: track 0.00 -> 255.4 mm
- net encA: track 0.00 -> 237.8 mm
- net encB: track 0.00 -> 229.8 mm
- net SDA: track 0.00 -> 210.6 mm, vias 0 -> 2
- net SCL: track 0.00 -> 202.3 mm, vias 0 -> 1
- net RotB: track 128.9 -> 327.1 mm
- net VCC: track 0.00 -> 181.4 mm
- net col4: track 165.4 -> 312.9 mm
- net col3: track 167.7 -> 279.7 mm
- net RotA: track 0.00 -> 77.9 mm, vias 0 -> 1
- net col2: track 153.1 -> 229.2 mm
- net RotC: track 0.00 -> 66.0 mm, vias 0 -> 2
- net rowH: track 123.2 -> 167.7 mm
- net col1: track 128.9 -> 169.5 mm
- net rowD: track 124.1 -> 156.8 mm
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Other:
- outline, holes or cut-outs redrawn

Commit message: Mounting holes and ground fill done
Parts:
- added REF**: MountingHole_2.2mm_M2, MountingHole:MountingHole_2.2mm_M2, F.Cu at (66.8, 105.0)
- added REF**: MountingHole_2.2mm_M2, MountingHole:MountingHole_2.2mm_M2, F.Cu at (62.1, 35.8)
- added REF**: MountingHole_2.2mm_M2, MountingHole:MountingHole_2.2mm_M2, F.Cu at (148.0, 66.8)
- added REF**: MountingHole_2.2mm_M2, MountingHole:MountingHole_2.2mm_M2, F.Cu at (229.2, 105.0)
- added REF**: MountingHole_2.2mm_M2, MountingHole:MountingHole_2.2mm_M2, F.Cu at (52.5, 66.8)
- added REF**: MountingHole_2.2mm_M2, MountingHole:MountingHole_2.2mm_M2, F.Cu at (243.5, 66.8)
- added REF**: MountingHole_2.2mm_M2, MountingHole:MountingHole_2.2mm_M2, F.Cu at (248.3, 35.8)
Routing:
- net col4: track 312.9 -> 317.3 mm
- net Net-(D45-Pad2): track 124.8 -> 128.4 mm
- net Net-(D36-Pad2): track 101.1 -> 104.6 mm
- net Net-(D24-Pad2): track 87.1 -> 90.3 mm
- net Net-(D42-Pad2): track 78.2 -> 81.2 mm
- net rowF: track 156.1 -> 158.8 mm
- net VCC: track 181.4 -> 183.7 mm
- net rowE: track 146.9 -> 148.9 mm
- net Net-(D31-Pad2): track 58.3 -> 60.3 mm
- net Net-(D43-Pad2): track 92.5 -> 94.5 mm
- net Net-(D38-Pad2): track 97.5 -> 98.5 mm
- net Net-(D44-Pad2): track 100.5 -> 101.3 mm
- net Net-(D20-Pad2): track 46.2 -> 46.9 mm
- added copper zone on B.Cu, net GND
- added copper zone on F.Cu, net GND
