File: litl_base_plate/litl_base_plate.kicad_pcb (KiCad board)
At the start: 2 copper layers, 254.3 x 105.9 mm, 13 parts

Commit message: Base and plates reworked
Parts:
- removed the REF** at (271.2, 129.9)
- removed the REF** at (54.6, 71.3)
- removed the REF** at (107.5, 129.9)
- removed the REF** at (150.1, 71.3)
- removed the REF** at (245.6, 71.3)
- removed the REF** at (189.4, 129.9)
- removed the REF** at (231.2, 109.5)
- removed the REF** at (68.9, 109.5)
- removed the REF** at (25.6, 56.7)
- removed the REF** at (25.6, 129.9)
- removed the REF** at (64.1, 40.2)
- removed the REF** at (271.2, 56.7)
- removed the REF** at (252.7, 40.2)
- added REF**: MountingHole_2.2mm_M2, MountingHole:MountingHole_2.2mm_M2, F.Cu at (23.9, 45.4)
- added REF**: MountingHole_2.2mm_M2, MountingHole:MountingHole_2.2mm_M2, F.Cu at (107.9, 119.4)
- added REF**: MountingHole_2.2mm_M2, MountingHole:MountingHole_2.2mm_M2, F.Cu at (189.7, 119.4)
- added REF**: MountingHole_4.3mm_M4, MountingHole:MountingHole_4.3mm_M4, F.Cu at (86.0, 45.4)
- added REF**: MountingHole_2.2mm_M2, MountingHole:MountingHole_2.2mm_M2, F.Cu at (276.9, 45.4)
- added REF**: MountingHole_2.2mm_M2, MountingHole:MountingHole_2.2mm_M2, F.Cu at (23.9, 119.4)
- added REF**: MountingHole_4.3mm_M4, MountingHole:MountingHole_4.3mm_M4, F.Cu at (214.9, 45.4)
- added REF**: MountingHole_2.2mm_M2, MountingHole:MountingHole_2.2mm_M2, F.Cu at (276.9, 119.4)
Routing:
- removed copper zone on F.Cu, net (none)
Other:
- board size 254.3 x 105.9 mm -> 262.6 x 107.4 mm
- board text added: "litl v1 design by mohoyt"

Commit message: Minimised base size and shrunk top of PCB to make it under 100mm. Send to fab
Routing:
- added copper zone on B.Cu, net (none)
- added copper zone on F.Cu, net (none)
Other:
- board text added: "JLCJLCJLCJLC"
- board text removed: "litl"
