File: litl_plate/litl_plate.kicad_pcb (KiCad board)
At the start: 2 copper layers, 254.3 x 82 mm, 11 parts

Commit message: Base and plates reworked
Parts:
- removed the REF** at (150.4, 76.4)
- removed the REF** at (245.9, 76.4)
- removed the REF** at (26.0, 135.0)
- removed the REF** at (231.6, 114.6)
- removed the REF** at (69.2, 114.6)
- removed the REF** at (107.9, 135.0)
- removed the REF** at (271.6, 61.8)
- removed the REF** at (189.7, 135.0)
- removed the REF** at (26.0, 61.8)
- removed the REF** at (54.9, 76.4)
- removed the REF** at (271.6, 135.0)
- added REF**: MountingHole_2.2mm_M2, MountingHole:MountingHole_2.2mm_M2, F.Cu at (24.0, 71.6)
- added REF**: MountingHole_2.2mm_M2, MountingHole:MountingHole_2.2mm_M2, F.Cu at (277.1, 145.6)
- added REF**: MountingHole_2.2mm_M2, MountingHole:MountingHole_2.2mm_M2, F.Cu at (108.0, 145.6)
- added REF**: MountingHole_2.2mm_M2, MountingHole:MountingHole_2.2mm_M2, F.Cu at (24.0, 145.6)
- added REF**: MountingHole_2.2mm_M2, MountingHole:MountingHole_2.2mm_M2, F.Cu at (189.8, 145.6)
- added REF**: MountingHole_2.2mm_M2, MountingHole:MountingHole_2.2mm_M2, F.Cu at (277.1, 71.6)
Routing:
- net (no net): vias 3 -> 4
Other:
- board size 254.3 x 82 mm -> 262.6 x 83.6 mm
- board text added: "litl v1 design by mohoyt"

Commit message: Minimised base size and shrunk top of PCB to make it under 100mm. Send to fab
Other:
- board text added: "JLCJLCJLCJLC"
Changed lines of the file:
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@@
       (layerselection 0x00010fc_ffffffff)
       (disableapertmacros false)
-      (usegerberextensions false)
+      (usegerberextensions true)
       (usegerberattributes true)
-      (usegerberadvancedattributes true)
-      (creategerberjobfile true)
+      (usegerberadvancedattributes false)
+      (creategerberjobfile false)
       (svguseinch false)
       (svgprecision 6)
@@
       (psa4output false)
       (plotreference true)
-      (plotvalue true)
+      (plotvalue false)
       (plotinvisibletext false)
       (sketchpadsonfab false)
-      (subtractmaskfromsilk false)
+      (subtractmaskfromsilk true)
       (outputformat 1)
       (mirror false)
-      (drillshape 1)
+      (drillshape 0)
       (scaleselection 1)
-      (outputdirectory "")
+      (outputdirectory "gerbers/")
     )
   )
@@
   (gr_line (start 34.02163 69.829581) (end 34.015097 69.853124) (layer "Edge.Cuts") (width 0.944881))
   (gr_line (start 133.654076 102.28171) (end 133.666103 102.260443) (layer "Edge.Cuts") (width 0.944881))
+  (gr_text "JLCJLCJLCJLC" (at 257.85 124.15) (layer "B.SilkS")
+    (effects (font (size 1 1) (thickness 0.15)) (justify mirror))
+  )
   (gr_text "litl v1\ndesign by mohoyt" (at 155.1875 105.05) (layer "B.SilkS")
     (effects (font (size 1 1) (thickness 0.15)) (justify mirror))
