File: PCB/litl_base/litl_base.kicad_pcb (KiCad board)
At the start: 2 copper layers, 262.6 x 83.6 mm, 8 parts

Commit message: V2 gerbers for production
Other:
- board text added: "litl v2 design by mohoyt"
- board text removed: "litl v1 design by mohoyt"
Changed lines of the file:
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@@
   (gr_line (start 23.875 59.6875) (end 276.95 59.6875) (layer "Edge.Cuts") (width 0.1))
   (gr_arc (start 276.95 59.6875) (mid 280.326435 61.086065) (end 281.725 64.4625) (layer "Edge.Cuts") (width 0.15))
-  (gr_text "litl v1\ndesign by mohoyt" (at 148.025 128.925) (layer "F.SilkS")
+  (gr_text "litl v2\ndesign by mohoyt" (at 148.025 128.925) (layer "F.SilkS")
     (effects (font (size 1 1) (thickness 0.15)))
   )

Commit message: Updated silkscreening on board and switch socket option added for encoders. Gerbers v2.1 added
Other:
- board text added: "STHLM KB litl v2 design by mohoyt"
- board text removed: "litl v2 design by mohoyt"
Changed lines of the file:
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@@
       (usegerberextensions true)
       (usegerberattributes true)
-      (usegerberadvancedattributes true)
-      (creategerberjobfile true)
+      (usegerberadvancedattributes false)
+      (creategerberjobfile false)
       (svguseinch false)
       (svgprecision 6)
@@
       (psnegative false)
       (psa4output false)
-      (plotreference false)
-      (plotvalue true)
+      (plotreference true)
+      (plotvalue false)
       (plotinvisibletext false)
       (sketchpadsonfab false)
@@
   (gr_line (start 23.875 59.6875) (end 276.95 59.6875) (layer "Edge.Cuts") (width 0.1))
   (gr_arc (start 276.95 59.6875) (mid 280.326435 61.086065) (end 281.725 64.4625) (layer "Edge.Cuts") (width 0.15))
-  (gr_text "litl v2\ndesign by mohoyt" (at 148.025 128.925) (layer "F.SilkS")
+  (gr_text "STHLM KB litl v2\ndesign by mohoyt" (at 148.025 128.925) (layer "F.SilkS")
     (effects (font (size 1 1) (thickness 0.15)))
   )
