File: PCB/litl_plate/litl_plate.kicad_pcb (KiCad board)
At the start: 2 copper layers, 262.6 x 83.6 mm, 6 parts

Commit message: V2 gerbers for production
Other:
- board text added: "litl v2 design by mohoyt"
- board text removed: "litl v1 design by mohoyt"

Commit message: Updated silkscreening on board and switch socket option added for encoders. Gerbers v2.1 added
Other:
- board text added: "STHLM KB litl v2 design by mohoyt"
- board text removed: "litl v2 design by mohoyt"
Changed lines of the file:
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@@
     (effects (font (size 1 1) (thickness 0.15)) (justify mirror))
   )
-  (gr_text "litl v2\ndesign by mohoyt" (at 155.1875 105.05) (layer "B.SilkS")
+  (gr_text "STHLM KB litl v2\ndesign by mohoyt" (at 155.1875 105.05) (layer "B.SilkS")
     (effects (font (size 1 1) (thickness 0.15)) (justify mirror))
   )
